File: keyboard.kicad_pcb (KiCad board)
At the start: 2 copper layers, 324.6 x 115.9 mm, 273 parts, among them J3 USB_C_Receptacle_USB2.0, Q1 DTC143Z, SW1 SW_Push, U1 MIC5219-3.3YMM, U3 STM32F072R8Tx, Y1 16MHz

Commit message: fixed led for minus with custom footprint
Parts:
- LED_minus1: renamed from LED_-1; footprint Keebio-Parts:SK6812-MINI-E -> keebio-Parts:SK6812-MINI-E-CUSTOM
- MX_6: footprint MX_Alps_Hybrid:MX-1U-NoLED -> pcb-guide:MX-1U-NoLED
- renumbered LED_\1 to LED_bs1, LED_,1 to LED_comma1, LED_=1 to LED_equal1, LED_/1 to LED_fs1, LED_.1 to LED_fullstop1, LED_[1 to LED_lb1, LED_'1 to LED_quote1, LED_]1 to LED_rb1, LED_;1 to LED_sc1
Routing:
- net +5V: track 1989.2 -> 1954.7 mm
- net ROW0: track 513.9 -> 514.5 mm

Commit message: Updated footprints, still need to do usb
Parts:
- ENC1: footprint eec:Bourns-PEC11R-4015F-S0024-MFG -> encoder:XDCR_PEC11R-4215F-S0024
- LED_0, LED_1, LED_2, LED_3, LED_4, LED_5, LED_6, LED_7, LED_8, LED_9, LED_A1, LED_B1, LED_BckSpace1, LED_C1, LED_CAPS1, LED_D1, LED_DOWN1, LED_Del1, LED_E1, LED_ENTER1, LED_End1, LED_Esc1, LED_F1, LED_F10, LED_F11, LED_F12, LED_F13, LED_F2, LED_F3, LED_F4, LED_F5, LED_F6, LED_F7, LED_F8, LED_F9, LED_G1, LED_H1, LED_Home1, LED_I1, LED_Ins1, LED_J1, LED_K1, LED_L1, LED_LALT1, LED_LCTRL1, LED_LEFT1, LED_LSHIFT1, LED_LWIN1, LED_M1, LED_N1, LED_O1, LED_P1, LED_PGDN1, LED_PGUP1, LED_PRTSCN1, LED_Q1, LED_R1, LED_RALT1, LED_RCTRL1, LED_RIGHT1, LED_RSHIFT1, LED_RWIN1, LED_S1, LED_SPACE1, LED_T1, LED_TAB1, LED_Tilda1, LED_U1, LED_UP1, LED_V1, LED_W1, LED_X1, LED_Y1, LED_Z1, LED_bs1, LED_comma1, LED_equal1, LED_fs1, LED_fullstop1, LED_lb1, LED_quote1, LED_rb1, LED_sc1: footprint Keebio-Parts:SK6812-MINI-E -> keebio-Parts:SK6812-MINI-E-CUSTOM
- MX_'1, MX_,1, MX_-1, MX_.1, MX_/1, MX_0, MX_1, MX_2, MX_3, MX_4, MX_5, MX_7, MX_8, MX_9, MX_;1, MX_=1, MX_A1, MX_B1, MX_C1, MX_D1, MX_Del1, MX_Down1, MX_E1, MX_End1, MX_Esc1, MX_F1, MX_F10, MX_F11, MX_F12, MX_F13, MX_F2, MX_F4, MX_F5, MX_F6, MX_F7, MX_F8, MX_F9, MX_G1, MX_H1, MX_Home1, MX_I1, MX_Ins1, MX_J1, MX_K1, MX_L1, MX_Left1, MX_M1, MX_N1, MX_O1, MX_P1, MX_PgDn1, MX_PgUp1, MX_PtrSc1, MX_Q1, MX_R1, MX_Right1, MX_S1, MX_T1, MX_Tilda1, MX_U1, MX_Up1, MX_V1, MX_W1, MX_X1, MX_Y1, MX_Z1, MX_[1, MX_]1: footprint MX_Alps_Hybrid:MX-1U-NoLED -> PCM_Switch_Keyboard_Cherry_MX:SW_Cherry_MX_PCB_1.00u
- MX_6: footprint pcb-guide:MX-1U-NoLED -> PCM_Switch_Keyboard_Cherry_MX:SW_Cherry_MX_PCB_1.00u
- MX_BckSpace1: footprint MX_Alps_Hybrid:MX-2U-NoLED -> PCM_Switch_Keyboard_Cherry_MX:Cherry 2u with stablizer
- MX_Caps1: footprint MX_Alps_Hybrid:MX-1.75U-NoLED -> PCM_Switch_Keyboard_Cherry_MX:SW_Cherry_MX_PCB_1.75u
- MX_Enter1, MX_LShift1: footprint MX_Alps_Hybrid:MX-2.25U-NoLED -> PCM_Switch_Keyboard_Cherry_MX:Cherry 2.25 with stablizer
- MX_F3: footprint MX_Alps_Hybrid:MX-1U-NoLED -> KiSwitch - Cherry Keyboard Switches:SW_Cherry_MX_PCB_1.00u
- MX_LAlt1, MX_LCtrl1, MX_LWin1, MX_RAlt1, MX_RCtrl1, MX_RWin1: footprint MX_Alps_Hybrid:MX-1.25U-NoLED -> PCM_Switch_Keyboard_Cherry_MX:SW_Cherry_MX_PCB_1.25u
- MX_RShift1: footprint MX_Alps_Hybrid:MX-2.75U-NoLED -> PCM_Switch_Keyboard_Cherry_MX:Cherry 2.75 with stablizer
- MX_Space1: footprint MX_Alps_Hybrid:MX-6U-Centered-NoLED -> PCM_Switch_Keyboard_Cherry_MX:Cherry 6u with upside down Stablizer
- MX_Tab1, MX_\1: footprint MX_Alps_Hybrid:MX-1.5U-NoLED -> PCM_Switch_Keyboard_Cherry_MX:SW_Cherry_MX_PCB_1.50u
Routing:
- net GND: track 2220.8 -> 2183.8 mm

Commit message: Updated usbc,moved leds,added gnd zone,fixed some routing
Parts:
- J3: footprint Connector_USB:USB_C_Receptacle_G-Switch_GT-USB-7010ASV -> usb_c:HRO_TYPE-C-31-M-12
- moved J3 0.95 mm to (50.4, 33.0)
- moved D73 0.25 mm to (277.1, 42.2)
- moved D10 0.16 mm to (81.9, 99.3)
- moved D5 0.16 mm to (53.3, 80.3)
- moved D15 0.16 mm to (96.2, 80.3)
- moved D16 0.16 mm to (101.0, 99.3)
- moved D21 0.16 mm to (115.3, 80.3)
- moved D22 0.16 mm to (120.0, 99.3)
- moved D27 0.16 mm to (134.3, 80.3)
- moved D28 0.16 mm to (139.1, 99.3)
- moved D33 0.16 mm to (153.4, 80.3)
- moved D34 0.16 mm to (158.1, 99.3)
- moved D39 0.16 mm to (172.4, 80.3)
- moved D40 0.16 mm to (177.2, 99.3)
- moved D45 0.16 mm to (191.5, 80.3)
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Connections:
- R5 pad 1: Net-(J3-CC1) -> GND
- R5 pad 2: GND -> Net-(J3-CC1)
Routing:
- net GND: track 2183.8 -> 22.2 mm, vias 16 -> 1
- net +5V: track 1954.7 -> 200.2 mm, vias 16 -> 15
- net COL15: track 237.3 -> 156.2 mm
- net Net-(LED_LALT1-DIN): track 64.6 -> 0.00 mm
- net ROW0: track 514.5 -> 457.0 mm
- net Net-(LED_RSHIFT1-DOUT): track 31.2 -> 0.00 mm
- net Net-(LED_RSHIFT1-DIN): track 31.2 -> 0.00 mm
- net Net-(LED_ENTER1-DIN): track 26.5 -> 0.00 mm
- net Net-(LED_LSHIFT1-DOUT): track 26.5 -> 0.00 mm
- net Net-(LED_LEFT1-DOUT): track 26.5 -> 0.00 mm
- net Net-(LED_ENTER1-DOUT): track 26.5 -> 0.00 mm
- net Net-(LED_A1-DOUT): track 21.7 -> 0.00 mm
- net Net-(LED_RCTRL1-DOUT): track 19.3 -> 0.00 mm
- net Net-(LED_RALT1-DIN): track 19.3 -> 0.00 mm
- net Net-(LED_LCTRL1-DIN): track 19.3 -> 0.00 mm
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- added copper zone on B.Cu, net GND
